Commit message: wip2

File: ros2_ws/src/tidybot_description/urdf/tidybot_wx250s.urdf.xacro (robot description, xacro)
@@ -55,5 +55,5 @@
     <parent link="base_link"/>
     <child link="camera_mount"/>
-    <origin xyz="0 -0.1125 0.279" rpy="0 0 -1.5708"/>
+    <origin xyz="0 -0.1125 0.279" rpy="0 0 0"/>
   </joint>
   <!-- ==================== PAN-TILT CAMERA SYSTEM ==================== -->

Commit message: fixed odom and base

File: ros2_ws/src/tidybot_description/urdf/tidybot_wx250s.urdf.xacro (robot description, xacro)
@@ -55,5 +55,5 @@
     <parent link="base_link"/>
     <child link="camera_mount"/>
-    <origin xyz="0 -0.1125 0.279" rpy="0 0 0"/>
+    <origin xyz="0 -0.1125 0.279" rpy="0 0 -1.5708"/>
   </joint>
   <!-- ==================== PAN-TILT CAMERA SYSTEM ==================== -->
